File: hardware/canpill.kicad_pcb (KiCad board)
At the start: 2 copper layers, 78 x 37 mm, 57 parts, among them J1 TYPE-C-31-M-12, J2 5100TR, J3 5100TR, J4 1776112-4, J5 Conn_01x20_Pin, J6 Conn_01x16_Pin, J7 FTSH-105-01-L-DV-K, SW1 SW_SPDT, SW2 SW_Push, U1 STM32F103C8T6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

Commit message: (software:canpill_test) initial commit; (hardware) add pull-up on DB_nRST
Parts:
- added R13: 10k, Resistor_SMD:R_0402_1005Metric, F.Cu at (121.2, 91.4)
